File: ergogen/output/pcbs/right.kicad_pcb (KiCad board)
At the start: 2 copper layers, 137 x 110 mm, 79 parts

Commit message: add switches and caps to ergogen output; not final pcb
Other:
- net class Default added: clearance 0.2, trace_width 0.25, via_dia 0.8, via_drill 0.4
